File: hardware/boards/osc-sg90-v006/osc-sg90-v006.kicad_pcb (KiCad board)
At the start: 4 copper layers, 20.6 x 9.6 mm, 34 parts, among them J1 Servo Input, J2 Motor, J3 Debug, J4 Potentiometer, M1 SG90_Motor, U1 H7133-1_C277537, U4 DRV8837, U5 CH32V006F8U6, U6 74LVC2G241GS,115

Commit message: update
Parts:
- added C5: 0.1µF, Capacitor_SMD:C_0402_1005Metric, F.Cu at (155.0, 85.0)
- added R10: TBD, Resistor_SMD:R_0402_1005Metric, F.Cu at (145.0, 85.0)
- added U7: ECC204-RBVCZ-T, shared:ECC204_Contact-3_L6.5-W2.5-P2.00, F.Cu at (150.0, 80.0)
Connections:
- U5 pad 20: unconnected-(U5-PD6/A6/RX/TX_1-Pad20) -> SE_SWIO
Changed lines of the file:
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@@
 			(size 0.2 0.8)
 			(layers "F.Cu" "F.Mask" "F.Paste")
-			(net "unconnected-(U5-PD6{slash}A6{slash}RX{slash}TX_1-Pad20)")
+			(net "SE_SWIO")
 			(pinfunction "PD6/A6/RX/TX_1_20")
-			(pintype "bidirectional+no_connect")
+			(pintype "bidirectional")
 		)
 		(pad "21" smd custom
@@
 		(layer "User.1")
 	)
+	(footprint "shared:ECC204_Contact-3_L6.5-W2.5-P2.00"
+		(layer "F.Cu")
+		(at 150 80)
+		(descr "Microchip ECC204 secure element, 3-Lead Contact (LAB/RHB), 6.54x2.5mm body, 2.0mm pitch [REF-SE-001 Sec 6.3]. STAGED -- not yet placed on board outline, see TODO.md Sec 7.8.")
+		(tags "secure-element ecc204 crypto")
+		(property "Reference" "U7"
+			(at 0 -2.2 0)
+			(layer "F.SilkS")
+			(hide yes)
+			(effects
+				(font
+					(size 1 1)
+					(thickness 0.15)
+				)
+			)
+		)
+		(property "Value" "ECC204-RBVCZ-T"
+			(at 0 2.2 0)
+			(layer "F.Fab")
+			(effects
+				(font
+					(size 1 1)
+					(thickness 0.15)
+				)
+			)
+		)
+		(sheetname "/")
+		(sheetfile "osc-sg90-v006.kicad_sch")
+		(attr smd)
+		(duplicate_pad_numbers_are_jumpers no)
+		(pad "1" smd rect
+			(at -2.0 0.0)
+			(size 1.8 2.3)
+			(layers "F.Cu" "F.Mask" "F.Paste")
+			(net "SE_SWIO")
+			(pintype "bidirectional")
+		)
+		(pad "2" smd rect
+			(at 0.0 0.0)
+			(size 1.8 2.3)
+			(layers "F.Cu" "F.Mask" "F.Paste")
+			(net "GND")
+			(pintype "power_in")
+		)
+		(pad "3" smd rect
+			(at 2.0 0.0)
+			(size 1.8 2.3)
+			(layers "F.Cu" "F.Mask" "F.Paste")
+			(net "+3V3")
+			(pintype "power_in")
+		)
+	)
+	(footprint "Resistor_SMD:R_0402_1005Metric"
+		(layer "F.Cu")
+		(at 145 85 180)
+		(descr "Resistor SMD 0402 (1005 Metric). SWI pull-up for U7 -- value TBD, see TODO.md Sec 7.4. STAGED -- not yet placed.")
+		(tags "resistor")
+		(property "Reference" "R10"
+			(at 0 -2.2 0)
+			(layer "F.SilkS")
+			(hide yes)
+			(effects
+				(font
+					(size 1 1)
+					(thickness 0.15)
+				)
+			)
+		)
+		(property "Value" "TBD"
+			(at 0 2.2 0)
+			(layer "F.Fab")
+			(effects
+				(font
+					(size 1 1)
+					(thickness 0.15)
+				)
+			)
+		)
+		(sheetname "/")
+		(sheetfile "osc-sg90-v006.kicad_sch")
+		(attr smd)
+		(duplicate_pad_numbers_are_jumpers no)
+		(pad "1" smd roundrect
+			(at -0.51 0)
+			(size 0.54 0.64)
+			(layers "F.Cu" "F.Mask" "F.Paste")
+			(roundrect_rratio 0.25)
+			(net "+3V3")
+			(pintype "passive")
+		)
+		(pad "2" smd roundrect
+			(at 0.51 0)
+			(size 0.54 0.64)
+			(layers "F.Cu" "F.Mask" "F.Paste")
+			(roundrect_rratio 0.25)
+			(net "SE_SWIO")
+			(pintype "passive")
+		)
+	)
+	(footprint "Capacitor_SMD:C_0402_1005Metric"
+		(layer "F.Cu")
+		(at 155 85)
+		(descr "Capacitor SMD 0402 (1005 Metric). VCC decoupling for U7. STAGED -- not yet placed.")
+		(tags "capacitor")
+		(property "Reference" "C5"
+			(at 0 -2.2 0)
+			(layer "F.SilkS")
+			(hide yes)
+			(effects
+				(font
+					(size 1 1)
+					(thickness 0.15)
+				)
+			)
+		)
+		(property "Value" "0.1µF"
+			(at 0 2.2 0)
+			(layer "F.Fab")
+			(effects
+				(font
+					(size 1 1)
+					(thickness 0.15)
+				)
+			)
+		)
+		(sheetname "/")
+		(sheetfile "osc-sg90-v006.kicad_sch")
+		(attr smd)
+		(duplicate_pad_numbers_are_jumpers no)
+		(pad "1" smd roundrect
+			(at -0.48 0)
+			(size 0.56 0.62)
+			(layers "F.Cu" "F.Mask" "F.Paste")
+			(roundrect_rratio 0.25)
+			(net "+3V3")
+			(pintype "passive")
+		)
+		(pad "2" smd roundrect
+			(at 0.48 0)
+			(size 0.56 0.62)
+			(layers "F.Cu" "F.Mask" "F.Paste")
+			(roundrect_rratio 0.25)
+			(net "GND")
+			(pintype "passive")
+		)
+	)
 	(gr_text "A"

Commit message: cleaned up a lot of stuff
Parts:
- removed the J4 at (115.8, 85.5)
- removed M1: SG90_Motor, shared:SG90_Motor
- removed REF**: SG90_Board_Outline, shared:SG90_Board_Outline
- C5, R10: moved to B.Cu
- U7: value ECC204-RBVCZ-T -> ECC204-MAVCZ-T; footprint shared:ECC204_Contact-3_L6.5-W2.5-P2.00 -> shared:ECC204_UDFN-8-1EP_L2.0-W3.0-P0.50-EP0.61x1.3mm; moved to B.Cu
- moved C5 55.3 mm to (101.0, 97.0)
- moved U7 51.0 mm to (101.3, 95.0), turned to 90 degrees
- moved R10 44.2 mm to (101.5, 93.0), turned to 0 degrees
- moved C10 3.10 mm to (103.0, 92.0)
- moved RS1 1.79 mm to (107.0, 97.1), turned to 180 degrees
- moved U1 0.10 mm to (107.2, 93.3)
- moved C2 0.08 mm to (108.2, 91.0)
Connections:
- U7 pad 1: SE_SWIO -> (no net)
- U7 pad 2: GND -> (no net)
- U7 pad 3: +3V3 -> (no net)
Routing:
- net /ISNS-: track 5.81 -> 1.35 mm, vias 1 -> 0
- net /ISNS+: track 4.80 -> 0.62 mm
- net VSYS: track 9.10 -> 5.40 mm, vias 2 -> 0
- net /SWDIO: track 3.14 -> 0.90 mm, vias 1 -> 0
- net /POT: track 3.96 -> 2.41 mm
- net /EN: track 4.08 -> 4.00 mm, vias 2 -> 1
- net PGND: vias 5 -> 4
Other:
- board size 20.6 x 9.6 mm -> 12.1 x 9.6 mm
